Commit message: frame transform

File: feldschwarm_robot_devel/urdf/feldschwarm_robot.gazebo.xacro (robot description, xacro)
@@ -45,6 +45,6 @@
       <alwaysOn>true</alwaysOn>
       <updateRate>50.0</updateRate>
-      <bodyName>chassis</bodyName>
-      <topicName>odom</topicName>
+      <bodyName>robot_footprint</bodyName>
+      <topicName>ground_truth/state</topicName>
       <gaussianNoise>0.01</gaussianNoise>
       <frameName>world</frameName>

File: feldschwarm_robot_devel/urdf/feldschwarm_robot.xacro (robot description, xacro)
@@ -257,5 +257,5 @@
   <xacro:include filename="$(find velodyne_description)/urdf/VLP-16.urdf.xacro"/>
   <VLP-16 parent="chassis" name="velodyne" topic="/velodyne_points" hz="10" samples="1024" gpu="false" lasers="16" max_range="100">
-    <origin xyz="0 0 0.4" rpy="0 0 0" />
+    <origin xyz="0 0 0.4" rpy="0 0 3.14  " />
   </VLP-16>
 </robot>

Commit message: update

File: feldschwarm_robot_devel/urdf/feldschwarm_robot.gazebo.xacro (robot description, xacro)
@@ -27,6 +27,6 @@
       <leftRearJoint>left_back_wheel_hinge</leftRearJoint>
       <rightRearJoint>right_back_wheel_hinge</rightRearJoint>
-      <wheelSeparation>0.46</wheelSeparation>
-      <wheelDiameter>0.16</wheelDiameter>
+      <wheelSeparation>0.01</wheelSeparation>
+      <wheelDiameter>0.2</wheelDiameter>
       <robotBaseFrame>robot_footprint</robotBaseFrame>
       <torque>200</torque>

File: feldschwarm_robot_devel/urdf/feldschwarm_robot.xacro (robot description, xacro)
@@ -5,5 +5,5 @@
   <xacro:property name="robot_width" value="${scale * 1}" />
   <xacro:property name="robot_length" value="${scale * 1.5}" />
-  <xacro:property name="robot_height" value="${scale * 0.4}" />
+  <xacro:property name="robot_height" value="${scale * 0.25}" />
   <xacro:property name="robot_mass" value="${scale * 20}" />
   <xacro:property name="base_x_offset" value="0" />
@@ -19,5 +19,5 @@
   <xacro:property name="robot_frame_height" value="${robot_height/4.0}" />
   <xacro:property name="wheel_length" value="${scale * 0.1}" />
-  <xacro:property name="wheel_radius" value="${scale * 0.2}" />
+  <xacro:property name="wheel_radius" value="${scale * 0.25}" />
   <xacro:property name="wheel_mass" value="${scale * 1}" />
   <xacro:property name="wheel_inertia" value="${scale * 1e-3}" />
@@ -31,6 +31,6 @@
   <xacro:property name="wheel_kp" value="1000000.0" />
   <xacro:property name="wheel_kd" value="100.0" />
-  <xacro:property name="wheel_mu1" value="1" />
-  <xacro:property name="wheel_mu2" value="1" />
+  <xacro:property name="wheel_mu1" value="0.8" />
+  <xacro:property name="wheel_mu2" value="0.8" />
   <xacro:property name="wheel_slip1" value="0.5" />
   <xacro:property name="wheel_slip2" value="0" />
